File: hardware/balancingFET.kicad_sch (KiCad schematic)
At the start: 5 parts

Commit message: init pcb
Parts:
- renumbered R9201 to R9101, R9101 to R9201

Commit message: update prj
Parts:
- gave numbers to parts that had none: 1
Other:
- company: (none) -> libreUPS
- title: (none) -> Balancer amplifier

Commit message: update readme
Parts:
- renumbered R9201 to R9101, R9101 to R9201

Commit message: update can
Parts:
- renumbered R9201 to R9101, R9101 to R9201
