File: hardware/main.kicad_sch (KiCad schematic)
At the start: 165 parts, among them J1 IDC-08M, J14 IDC-08M, J15 DS1013-10S, J2 B3B-XH-A, J4 IDC-08M, J5 B2B-XH-A, J6 B2B-XH-A, J8 XT60, J9 XT60, Q1 5N10-MS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

Commit message: fix prj; description -> Comments
Parts:
- Q1, Q2: Comments (none) -> bss123; description bss123 -> (none)
- U3: Comments (none) -> ISO1050DUB; description ISO1050DUB -> (none)
Changed lines of the file:
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@@
       (effects (font (size 1.27 1.27)) hide)
     )
-    (property "description" "bss123" (at 237.49 105.41 0)
+    (property "Comments" "bss123" (at 237.49 105.41 0)
       (effects (font (size 1.27 1.27)) hide)
     )
@@
       (effects (font (size 1.27 1.27)) hide)
     )
-    (property "description" "bss123" (at 327.66 85.09 0)
+    (property "Comments" "bss123" (at 327.66 85.09 0)
       (effects (font (size 1.27 1.27)) hide)
     )
@@
       (effects (font (size 1.27 1.27)) hide)
     )
-    (property "description" "ISO1050DUB" (at 247.65 49.53 0)
+    (property "Comments" "ISO1050DUB" (at 247.65 49.53 0)
       (effects (font (size 1.27 1.27)) hide)
     )
