File: hardware/main.kicad_sch (KiCad schematic)
At the start: 164 parts, among them SW1 TS-1187A-B-A-B, U1 TPS54360BDDx, U3101 AM1LS-0505S-NZ, U5 LM1117GS-3.3 (!)

Commit message: finish sch
Parts:
- removed C15: 100u, Capacitor_Tantalum_SMD:CP_EIA-7343-31_Kemet-D, symbol Device:C_Polarized_Small
- removed C15: 10u, Capacitor_Tantalum_SMD:CP_EIA-7343-31_Kemet-D, symbol Device:C_Polarized_Small
- removed C15 (x2): 22u, Capacitor_Tantalum_SMD:CP_EIA-7343-43_Kemet-X, symbol Device:C_Polarized_Small
- removed C4: 100n, Capacitor_SMD:C_0805_2012Metric, symbol Device:C_Small
- removed C52: 6.8n, Capacitor_SMD:C_0603_1608Metric, symbol Device:C_Small
- removed C52: 39p, Capacitor_SMD:C_0603_1608Metric, symbol Device:C_Small
- removed C80 (x2), C86 (x2): 22u, Capacitor_SMD:C_0805_2012Metric, symbol Device:C_Small
- removed C? (x4): 100n, Capacitor_SMD:C_0603_1608Metric, symbol Device:C_Small
- removed C?: 1n, Capacitor_SMD:C_0603_1608Metric, symbol Device:C_Small
- removed C? (x3): 2.2u, Capacitor_SMD:C_1206_3216Metric, symbol Device:C_Small
- removed C?: 330p, Capacitor_SMD:C_0603_1608Metric, symbol Device:C_Small
- removed C?: 100n, MAS_Package_nostd:B32652A3474J000, symbol Device:C_Small
- removed D23: BZV55C10, Diode_SMD:D_MiniMELF, symbol Device:D_Zener
- removed D5, D?: LED_yellow, LED_SMD:LED_0603_1608Metric, symbol Device:LED_Small
- removed D?: SMBJ54A, Diode_SMD:D_SMB, symbol Device:D_Zener_Small
- removed F?: S1032-F-40.0A, MAS_Package_nostd:Fuse_1032, symbol Device:Fuse_Small
- removed H3: H, MountingHole:MountingHole_3.2mm_M3_DIN965_Pad, symbol Mechanical:MountingHole
- removed J? (x3): XT60, MAS_Package_nostd:AMASS_XT60-F_1x02_P7.20mm_Vertical, symbol MAS_Connectors:XT60
- removed J?: 98424-G52-08ALF, MAS_Package_std:PinSocket_2x04_P2.00mm_Vertical_SMD, symbol Connector_Generic:Conn_02x04_Odd_Even
- removed JP3: div1, MAS_Package_nostd:SolderJumper_Open_Pad0.5x0.8mm, symbol Jumper:Jumper_2_Open
- removed JP?: A1, MAS_Package_nostd:SolderJumper_Open_Pad0.5x0.8mm, symbol Jumper:Jumper_2_Open
- removed JP?: A0, MAS_Package_nostd:SolderJumper_Open_Pad0.5x0.8mm, symbol Jumper:Jumper_2_Open
- removed R32: 1k, Resistor_SMD:R_0603_1608Metric, symbol Device:R_Small
- removed R32: 2.2k, Resistor_SMD:R_0603_1608Metric, symbol Device:R_Small
- removed R9101: 10k, Resistor_SMD:R_0603_1608Metric, symbol Device:R_Small
- removed R9102: 4.7k, Resistor_SMD:R_0603_1608Metric, symbol Device:R_Small
- removed R9103: 10R, Resistor_SMD:R_0603_1608Metric, symbol Device:R_Small
- removed R?: 13k, Resistor_SMD:R_0603_1608Metric, symbol Device:R_Small
- removed R? (x6): 430k, Resistor_SMD:R_0805_2012Metric, symbol Device:R_Small
- removed R?: 100k, Resistor_SMD:R_0805_2012Metric, symbol Device:R_Small
- removed R? (x3): 10R, Resistor_SMD:R_0402_1005Metric, symbol Device:R_Small
- removed R?: 1k, Resistor_SMD:R_0402_1005Metric, symbol Device:R_Small
- removed R?: 27k, Resistor_SMD:R_0603_1608Metric, symbol Device:R_Small
- removed R? (x2): 4.7k, Resistor_SMD:R_0402_1005Metric, symbol Device:R_Small
- removed R?: 220R, Resistor_SMD:R_0402_1005Metric, symbol Device:R_Small
- removed R? (x3): 0.5m, Resistor_SMD:R_2512_6332Metric, symbol Device:R_Small
- removed R?: 162k, Resistor_SMD:R_0603_1608Metric, symbol Device:R_Small
- removed U1: TPS54360BDDx, MAS_Package_std:Texas_R-PDSO-G8_EP2.95x4.9mm_Mask2.4x3.1mm, symbol MAS_IC_PowerSupply:TPS54360
- removed U5: LM1117GS-3.3 (!), Package_TO_SOT_SMD:SOT-223-3_TabPin2, symbol Regulator_Linear:LM1117-3.3
- removed U?: INA226, Package_SO:VSSOP-10_3x3mm_P0.5mm, symbol Sensor_Energy:INA226
- added C45 (x4): 12p, Capacitor_SMD:C_0603_1608Metric, symbol Device:C_Small
- added C52 (x11): 100n, Capacitor_SMD:C_0603_1608Metric, symbol Device:C_Small
- added C80, C86: 22u, Capacitor_SMD:C_0805_2012Metric, symbol Device:C_Small
- added C? (x2): 2.2u, Capacitor_SMD:C_1206_3216Metric, symbol Device:C_Small
- added C? (x2): 330p, Capacitor_SMD:C_0603_1608Metric, symbol Device:C_Small
- added C? (x2): 100n, Capacitor_SMD:C_1206_3216Metric, symbol Device:C_Small
- added D2 (x3): BZT52C3V3, Diode_SMD:D_SOD-323, symbol Device:D_Small
- added D2: 1N4148WS, Diode_SMD:D_SOD-323, symbol Device:D_Small
- added D2: STPS2L40U, Diode_SMD:D_SMB, symbol Device:D_Small
- added F?: S1032-F-40.0A, MAS_Package_nostd:Fuse_1032, symbol Device:Fuse_Small
- added J14: IDC-08M, Connector_IDC:IDC-Header_2x04_P2.54mm_Vertical, symbol Connector_Generic:Conn_02x04_Counter_Clockwise
- added J15: DS1013-10S, Connector_IDC:IDC-Header_2x05_P2.54mm_Vertical, symbol Connector_Generic:Conn_02x05_Odd_Even
- added J? (x3): B2B-XH-A, MAS_Package_std:JST_XH_B2B-XH-AM_1x02_P2.50mm_Vertical, symbol Connector_Generic:Conn_01x02
- added J? (x2): HC-MX3.0-2*4A, MAS_Package_std:Molex_Micro-Fit_3.0_43045-0812_2x04_P3.00mm_Vertical, symbol Connector_Generic:Conn_02x04_Top_Bottom
- added JP3 (x2): div1, MAS_Package_nostd:SolderJumper_Open_Pad0.5x0.8mm, symbol Jumper:Jumper_2_Open
- added JP?: Jload, MAS_Package_nostd:SolderJumper_Open_Pad0.5x0.8mm, symbol Jumper:Jumper_2_Open
- added Q?: 5N10-MS, Package_TO_SOT_SMD:SOT-23, symbol Transistor_FET:2N7002
- added R9101 (x4): 100R, Resistor_SMD:R_0603_1608Metric, symbol Device:R_Small
- added R9101 (x2): 100k, Resistor_SMD:R_0603_1608Metric, symbol Device:R_Small
- added R9101 (x2): 0R, Resistor_SMD:R_0603_1608Metric, symbol Device:R_Small
- added R9101: 1k, Resistor_SMD:R_0603_1608Metric, symbol Device:R_Small
- added R9101: 51k, Resistor_SMD:R_0603_1608Metric, symbol Device:R_Small
- added R9101, R9201 (x3): 4.7k, Resistor_SMD:R_0603_1608Metric, symbol Device:R_Small
- added R9105: 120R, Resistor_SMD:R_1206_3216Metric, symbol Device:R_Small
- added R? (x2): 3m, Resistor_SMD:R_2512_6332Metric, symbol Device:R_Small
- added R?: 10k/NTC, Resistor_SMD:R_0603_1608Metric, symbol MAS_Resistors:Thermistor_NTC
- added R?: 18k, Resistor_SMD:R_0603_1608Metric, symbol Device:R_Small
- added R?: 47k, Resistor_SMD:R_0603_1608Metric, symbol Device:R_Small
- added U?: LMR16030SDDAR, MAS_Package_std:SOIC-8-1EP_3.9x4.9mm_P1.27mm_EP2.29x3mm, symbol MAS_IC_PowerSupply:LMR16030
- added Y1: NX3215SA-32.768, MAS_Package_std:Crystal_SMD_3215-2Pin_3.2x1.5mm, symbol Device:Crystal
- added Y1: X50328MSB2GI, MAS_Package_std:Crystal_SMD_5032-2Pin_5.0x3.2mm, symbol Device:Crystal
- D2: value BZT52C5V6S -> BZT52C3V3; lcsc C2891792 -> C2932735
- J?: now fitted
- R?: value 5.1k -> 18k; lcsc C23186 -> C25810
- TP?: value SDA -> SCL
- TP?: value SCL -> SDA
- renumbered R9201 to R9101
Connections:
- net REGOUT is gone; now on net +3.3V: C80.1, R9101.2, R9101.2, U?.8 (REGOUT)
- net +3.3V: now also U?.1 (VCC1), U?.24 (VDD), U?.36 (VDD), U?.48 (VDD), U?.9 (VDDA), C52.1, C52.1, C52.1, C52.1, C52.1, C52.1, C52.1, JP3.2 (B), JP3.2 (B), R9101.2, R9201.2
- net +5V: now also U3101.2 (+Vin), C52.1, C52.1, C86.1, D2.1 (K), J?.1 (Pin_1), R9101.1
- net ALERT: now also U?.41 (PB5)
- net B1: now also R9101.2; no longer SW1.2
- net BAT+: now also C?.1, D3102.1 (K), D?.1 (A1), F1.2, C?.1, F?.2, J?.8 (Pin_8)
- net C1: now also J?.2 (Pin_2)
- net C10: now also J?.3 (Pin_3)
- net C11: now also J?.4 (Pin_4)
- net C12: now also J?.5 (Pin_5)
- net C13: now also J?.6 (Pin_6)
- net C14: now also J?.7 (Pin_7)
- net C2: now also J?.3 (Pin_3)
- net C3: now also J?.4 (Pin_4)
- net C4: now also J?.5 (Pin_5)
- net C5: now also J?.6 (Pin_6)
- net C6: now also J?.7 (Pin_7)
- net C7: now also J?.8 (Pin_8)
- net C8: now also J?.1 (Pin_1)
- net C9: now also J?.2 (Pin_2)
- net GND: now also C?.2, U3101.1 (-Vin), U?.23 (VSS), U?.35 (VSS), U?.4 (GND1), U?.47 (VSS), U?.8 (VSSA), C45.2, C45.2, C45.2, C45.2, C52.2, C52.2, C52.2, C52.2, C52.2, C52.2, C52.2, C52.2, C52.2, C52.2, C86.2, C?.2, C?.2, C?.2, D2.2 (A), D2.2 (A), D2.2 (A), J14.1 (Pin_1), J15.6 (Pin_6), J?.1 (Pin_1), Q?.2 (S), R9101.1, R9101.1, R9201.1, R?.1, R?.1, R?.2, R?.2, R?.2, U?.7 (GND), U?.9 (GND)
- net PACK+: now also F?.1; no longer C?.1, D3102.1 (K), D?.1 (A1)
- net SCL: now also TP?.1, U?.42 (PB6)
- net SDA: now also TP?.1, U?.43 (PB7)
- net SRN: now also D2.1 (K)
- net SRP: now also D2.1 (K)
- net VC10x: now also J?.2 (Pin_2)
- net VC5x: now also J?.2 (Pin_2)
- net V_BAT: now also U?.10 (PA0)
- net at F1.1: now also C?.1, C?.1, C?.1, U?.2 (VIN)
- net at C52.1: now also U?.1 (BOOT)
- net at R?.2: now also R9101.2, U?.5 (FB)
- net at C52.2, D2.1 (K), L1.1: now also U?.8 (SW)
- net at C?.1, U?.6 (TS1): now also R9201.1, R?.1
- net at D9101.1 (K): now also U?.6 (CANL), R9101.1, R9101.2, R9105.2
- net at D9101.2 (K): now also R9101.1, U?.7 (CANH), JP?.2 (B), R9101.1
- net CANgnd: now reaches D9101.3 (A)
- net CANgnd: now also U3101.4 (-Vout), U?.5 (GND2), C52.2, C80.2, C?.2, C?.2, J15.9 (Pin_9)
- net at C?.2, U?.18 (TS3): now also J?.1 (Pin_1)
- net at C?.1, Q?.2 (S), R9101.1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: now also R?.1, R?.1
- net K2: now reaches SW1.1
- net K2: now also D2.2 (A), J15.2 (Pin_2), R9101.1
- net at C?.1, U?.13 (TS2): now also J?.1 (Pin_1)
- net at U?.1 (VBAT): now also R9101.1
- net LSE_IN: now reaches U?.14 (PA4)
- net LSE_IN: now also C45.1, Y1.1
- net LSE_OUT: now reaches U?.15 (PA5)
- net LSE_OUT: now also C45.1, Y1.2
- net IO1: now reaches U?.25 (PB12)
- net IO1: now also J15.3 (Pin_3)
- net IO2: now reaches U?.26 (PB13)
- net IO2: now also J15.4 (Pin_4)
- net IO3: now reaches U?.27 (PB14)
- net IO3: now also J15.5 (Pin_5)
- net IO4: now reaches U?.28 (PB15)
- net IO4: now also R9101.2
- net DBG_TX: now reaches U?.30 (PA9)
- net DBG_TX: now also J14.6 (Pin_6)
- net DBG_RX: now reaches U?.31 (PA10)
- net DBG_RX: now also J14.5 (Pin_5)
- net CANrx: now reaches U?.32 (PA11)
- net CANrx: now also U?.2 (RXD)
- net CANtx: now reaches U?.33 (PA12)
- net CANtx: now also U?.3 (TXD)
- net SYS_SWDIO: now reaches U?.34 (PA13)
- net SYS_SWDIO: now also J14.3 (Pin_3)
- net SYS_SWCLK: now reaches U?.37 (PA14)
- net SYS_SWCLK: now also J14.4 (Pin_4)
- net EN5V: now reaches U?.38 (PA15)
- net EN5V: now also R9101.2
- net SYS_SWO: now reaches U?.39 (PB3)
- net SYS_SWO: now also J14.2 (Pin_2)
- net BTN: now reaches U?.40 (PB4)
- net BTN: now also D2.1 (K), R9101.2, R9101.2
- net BOOT0: now reaches U?.44 (BOOT0)
- net BOOT0: now also JP3.1 (A), R9201.2
- net HSE_IN: now reaches U?.5 (PD0)
- net HSE_IN: now also C45.1, Y1.1
- net HSE_OUT: now reaches U?.6 (PD1)
- net HSE_OUT: now also C45.1, Y1.2
- net NRST: now reaches U?.7 (NRST)
- net NRST: now also C52.1, J14.7 (Pin_7), R9201.1
- net CANvcc: now reaches U3101.5 (+Vout)
- net CANvcc: now also U?.8 (VCC2), C52.1, C80.1, J15.10 (Pin_10)
- net at R9101.2: now also C?.1
- new net: J14.8 (Pin_8), JP3.1 (A)
- new net: D2.1 (K), R9201.2
- new net: C?.1, C?.2
- new net: R9101.1, U?.3 (EN)
- new net: R?.2, U?.4 (RT/CLK)
- new net: R?.2, U?.6 (SS/PG)
- new net: D2.2 (A), J?.2 (Pin_2), Q?.3 (D)
- new net: Q?.1 (G), R9101.1, R9101.2
- new net: JP?.1 (A), R9105.1
- new net: C?.1, R9101.2
- new net CANH: J15.7 (Pin_7), R9101.2
- new net CANL: J15.8 (Pin_8), R9101.1
- new net K1: J15.1 (Pin_1), R9101.1, SW1.2
Other:
- note removed: "V: +1000v C: 100A"
- moved on the sheet: C4, C52, C80, C86, C?, D2, D9101, D?, F1, L1, Q?, R9101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

Commit message: init pcb
Parts:
- renumbered R9201 to R9101, R9101 to R9201

Commit message: update prj
Parts:
- D2: value STPS2L40U -> MBR0540; footprint Diode_SMD:D_SMB -> Diode_SMD:D_SOD-123; chipdip 2666823191 -> 9000072378; lcsc C169095 -> C699113; promelec 126735 -> 112220
- gave numbers to parts that had none: 19
Connections:
- net BAT+: now also J8.2
- net GND: now also J8.1
- net PACK+: now also J9.2
- net PACK-: now also J9.1
Other:
- company: (none) -> libreUPS
- title: (none) -> Battery management system
- moved on the sheet: C4, C45, C52, C80, C86, C?, D10, D2, D3102, D9101, F1, F2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

Commit message: update pcb
Parts:
- J14: footprint Connector_IDC:IDC-Header_2x04_P2.54mm_Vertical -> Connector_PinSocket_1.27mm:PinSocket_2x04_P1.27mm_Vertical
- JP3: value div1 -> PWRprog
- JP3: value div1 -> BOOT
Changed lines of the file:
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@@
       (effects (font (size 1.27 1.27)))
     )
-    (property "Value" "div1" (at 389.89 173.8884 0)
+    (property "Value" "PWRprog" (at 389.89 173.8884 0)
       (effects (font (size 1.27 1.27)) hide)
     )
@@
       )
       (project "main"
+        (path "/fa2fe869-55e7-4e89-bcf2-910d5ca003e8/9281d2dd-47ae-4ece-8b7d-5f799815d8f6"
+          (reference "D?") (unit 1)
+        )
         (path "/fa2fe869-55e7-4e89-bcf2-910d5ca003e8"
           (reference "D11") (unit 1)
@@
           (reference "D?") (unit 1)
         )
-        (path "/fa2fe869-55e7-4e89-bcf2-910d5ca003e8/79027519-9adf-41e5-b477-509d06c88a64"
-          (reference "D?") (unit 1)
-        )
         (path "/fa2fe869-55e7-4e89-bcf2-910d5ca003e8/804a2ff5-fd9a-4bb9-b248-5c8764c099f2"
           (reference "D?") (unit 1)
         )
-        (path "/fa2fe869-55e7-4e89-bcf2-910d5ca003e8/9281d2dd-47ae-4ece-8b7d-5f799815d8f6"
-          (reference "D?") (unit 1)
-        )
         (path "/fa2fe869-55e7-4e89-bcf2-910d5ca003e8/7363d190-73c2-4872-af97-478bf4c0edb0"
           (reference "D?") (unit 1)
@@
           (reference "D?") (unit 1)
         )
+        (path "/fa2fe869-55e7-4e89-bcf2-910d5ca003e8/79027519-9adf-41e5-b477-509d06c88a64"
+          (reference "D?") (unit 1)
+        )
       )
     )
@@
       (effects (font (size 1.27 1.27)))
     )
-    (property "Footprint" "Connector_IDC:IDC-Header_2x04_P2.54mm_Vertical" (at 374.65 180.34 0)
+    (property "Footprint" "Connector_PinSocket_1.27mm:PinSocket_2x04_P1.27mm_Vertical" (at 374.65 180.34 0)
       (effects (font (size 1.27 1.27)) hide)
     )
@@
       )
       (project "main"
+        (path "/fa2fe869-55e7-4e89-bcf2-910d5ca003e8/9281d2dd-47ae-4ece-8b7d-5f799815d8f6"
+          (reference "D?") (unit 1)
+        )
         (path "/fa2fe869-55e7-4e89-bcf2-910d5ca003e8"
           (reference "D12") (unit 1)
@@
           (reference "D?") (unit 1)
         )
-        (path "/fa2fe869-55e7-4e89-bcf2-910d5ca003e8/79027519-9adf-41e5-b477-509d06c88a64"
-          (reference "D?") (unit 1)
-        )
         (path "/fa2fe869-55e7-4e89-bcf2-910d5ca003e8/804a2ff5-fd9a-4bb9-b248-5c8764c099f2"
           (reference "D?") (unit 1)
         )
-        (path "/fa2fe869-55e7-4e89-bcf2-910d5ca003e8/9281d2dd-47ae-4ece-8b7d-5f799815d8f6"
-          (reference "D?") (unit 1)
-        )
         (path "/fa2fe869-55e7-4e89-bcf2-910d5ca003e8/7363d190-73c2-4872-af97-478bf4c0edb0"
           (reference "D?") (unit 1)
@@
           (reference "D?") (unit 1)
         )
+        (path "/fa2fe869-55e7-4e89-bcf2-910d5ca003e8/79027519-9adf-41e5-b477-509d06c88a64"
+          (reference "D?") (unit 1)
+        )
       )
     )
@@
       )
       (project "main"
+        (path "/fa2fe869-55e7-4e89-bcf2-910d5ca003e8/9f77eeed-fe35-4a84-a133-e30ed053e6d2"
+          (reference "D?") (unit 1)
+        )
         (path "/fa2fe869-55e7-4e89-bcf2-910d5ca003e8/bdc2dd95-da21-4e41-b835-133194d0a27b"
           (reference "D?") (unit 1)
@@
           (reference "D15") (unit 1)
         )
-        (path "/fa2fe869-55e7-4e89-bcf2-910d5ca003e8/4518093f-f1f9-4c04-81d1-07b4e3318740"
-          (reference "D?") (unit 1)
-        )
         (path "/fa2fe869-55e7-4e89-bcf2-910d5ca003e8/804a2ff5-fd9a-4bb9-b248-5c8764c099f2"
           (reference "D?") (unit 1)
         )
-        (path "/fa2fe869-55e7-4e89-bcf2-910d5ca003e8/9f77eeed-fe35-4a84-a133-e30ed053e6d2"
-          (reference "D?") (unit 1)
-        )
         (path "/fa2fe869-55e7-4e89-bcf2-910d5ca003e8/79027519-9adf-41e5-b477-509d06c88a64"
           (reference "D?") (unit 1)
@@
           (reference "D?") (unit 1)
         )
+        (path "/fa2fe869-55e7-4e89-bcf2-910d5ca003e8/4518093f-f1f9-4c04-81d1-07b4e3318740"
+          (reference "D?") (unit 1)
+        )
       )
     )
@@
       )
       (project "main"
+        (path "/fa2fe869-55e7-4e89-bcf2-910d5ca003e8/9281d2dd-47ae-4ece-8b7d-5f799815d8f6"
+          (reference "D?") (unit 1)
+        )
         (path "/fa2fe869-55e7-4e89-bcf2-910d5ca003e8"
           (reference "D9") (unit 1)
@@
           (reference "D?") (unit 1)
         )
-        (path "/fa2fe869-55e7-4e89-bcf2-910d5ca003e8/79027519-9adf-41e5-b477-509d06c88a64"
-          (reference "D?") (unit 1)
-        )
         (path "/fa2fe869-55e7-4e89-bcf2-910d5ca003e8/804a2ff5-fd9a-4bb9-b248-5c8764c099f2"
           (reference "D?") (unit 1)
         )
-        (path "/fa2fe869-55e7-4e89-bcf2-910d5ca003e8/9281d2dd-47ae-4ece-8b7d-5f799815d8f6"
-          (reference "D?") (unit 1)
-        )
         (path "/fa2fe869-55e7-4e89-bcf2-910d5ca003e8/7363d190-73c2-4872-af97-478bf4c0edb0"
           (reference "D?") (unit 1)
@@
           (reference "D?") (unit 1)
         )
+        (path "/fa2fe869-55e7-4e89-bcf2-910d5ca003e8/79027519-9adf-41e5-b477-509d06c88a64"
+          (reference "D?") (unit 1)
+        )
       )
     )
@@
       )
       (project "main"
+        (path "/fa2fe869-55e7-4e89-bcf2-910d5ca003e8/9281d2dd-47ae-4ece-8b7d-5f799815d8f6"
+          (reference "D?") (unit 1)
+        )
         (path "/fa2fe869-55e7-4e89-bcf2-910d5ca003e8"
           (reference "D16") (unit 1)
@@
           (reference "D?") (unit 1)
         )
-        (path "/fa2fe869-55e7-4e89-bcf2-910d5ca003e8/79027519-9adf-41e5-b477-509d06c88a64"
-          (reference "D?") (unit 1)
-        )
         (path "/fa2fe869-55e7-4e89-bcf2-910d5ca003e8/804a2ff5-fd9a-4bb9-b248-5c8764c099f2"
           (reference "D?") (unit 1)
         )
-        (path "/fa2fe869-55e7-4e89-bcf2-910d5ca003e8/9281d2dd-47ae-4ece-8b7d-5f799815d8f6"
-          (reference "D?") (unit 1)
-        )
         (path "/fa2fe869-55e7-4e89-bcf2-910d5ca003e8/7363d190-73c2-4872-af97-478bf4c0edb0"
           (reference "D?") (unit 1)
@@
           (reference "D?") (unit 1)
         )
+        (path "/fa2fe869-55e7-4e89-bcf2-910d5ca003e8/79027519-9adf-41e5-b477-509d06c88a64"
+          (reference "D?") (unit 1)
+        )
       )
     )
@@
       (effects (font (size 1.27 1.27)))
     )
-    (property "Value" "div1" (at 361.8484 105.41 0)
+    (property "Value" "BOOT" (at 361.8484 105.41 0)
       (effects (font (size 1.27 1.27)) hide)
     )

Commit message: update readme
Parts:
- removed J2: B2B-XH-A, MAS_Package_std:JST_XH_B2B-XH-AM_1x02_P2.50mm_Vertical, symbol Connector_Generic:Conn_01x02
- added J2: B3B-XH-A, MAS_Package_std:JST_XH_B3B-XH-AM_1x03_P2.50mm_Vertical, symbol Connector_Generic:Conn_01x03
- J1, J4: value HC-MX3.0-2*4A -> IDC-08M; footprint MAS_Package_std:Molex_Micro-Fit_3.0_43045-0812_2x04_P3.00mm_Vertical -> Connector_IDC:IDC-Header_2x04_P2.54mm_Vertical; chipdip (none) -> 9000376904; lcsc C3294373 -> C358742
Connections:
- net +5V: now also J2.1 (Pin_1)
- net GND: now also J2.3 (Pin_3)
- net at D2.2 (A), Q1.3 (D): now also J2.2 (Pin_2)

Commit message: update can
Parts:
- removed C52 (x3): 100n, Capacitor_SMD:C_0603_1608Metric, symbol Device:C_Small
- removed C80, C86: 22u, Capacitor_SMD:C_0805_2012Metric, symbol Device:C_Small
- removed C? (x2): 330p, Capacitor_SMD:C_0603_1608Metric, symbol Device:C_Small
- removed JP?: Jload, MAS_Package_nostd:SolderJumper_Open_Pad0.5x0.8mm, symbol Jumper:Jumper_2_Open
- removed R9101 (x2): 0R, Resistor_SMD:R_0603_1608Metric, symbol Device:R_Small
- removed R9101 (x2): 100R, Resistor_SMD:R_0603_1608Metric, symbol Device:R_Small
- removed U3: CA-IS3050G, MAS_Package_std:SOIC-8_7.5x5.85mm_P1.27mm, symbol MAS_IC_Interface:CA-IS305xG
- removed U3101: AM1LS-0505S-NZ, MAS_Package_nostd:Converter_DCDC_Aimtec_AM1LS_SMD, symbol MAS_Module:AM1LS-0505S-NZ
- added C52 (x2): 10u, Capacitor_SMD:C_0603_1608Metric, symbol Device:C_Small
- added C9102: 1n (-), Capacitor_SMD:C_1206_3216Metric, symbol Device:C_Small
- added C? (x2): 330p, Capacitor_SMD:C_0603_1608Metric, symbol Device:C_Small
- added C? (x2): 100n, Capacitor_SMD:C_0603_1608Metric, symbol Device:C_Small
- added D2: MBR0540, Diode_SMD:D_SOD-123, symbol Device:D_Small
- added J10: B3B-XH-A, MAS_Package_std:JST_XH_B3B-XH-AM_1x03_P2.50mm_Vertical, symbol Connector_Generic:Conn_01x03
- added JP?: Jload, MAS_Package_nostd:SolderJumper_Open_Pad0.5x0.8mm, symbol Jumper:Jumper_2_Open
- added Q21: 5N10-MS, Package_TO_SOT_SMD:SOT-23, symbol Transistor_FET:2N7002
- added R9101: 100k, Resistor_SMD:R_0603_1608Metric, symbol Device:R_Small
- added R9101 (x2): 0R, Resistor_SMD:R_0603_1608Metric, symbol Device:R_Small
- added R9101 (x3): 100R, Resistor_SMD:R_0603_1608Metric, symbol Device:R_Small
- added U1: CA-IS3062W, Package_SO:SOIC-16W_7.5x10.3mm_P1.27mm, symbol MAS_IC_Interface:CA-IS3062W
Connections:
- net +3.3V: now also C52.1, C?.1, U1.1 (VDD1)
- net +5V: now also D2.1 (K), J10.1 (Pin_1)
- net CANH: now also R9101.1
- net CANL: now also R9101.1
- net CANgnd: now also C52.2, C9102.2, C?.2, C?.2, C?.2, U1.10 (GND2), U1.15 (GND2), U1.9 (GND2)
- net CANrx: now also U1.5 (RxD)
- net CANtx: now also U1.3 (TxD)
- net CANvcc: now also C52.1, C?.1, U1.11 (VDD2), U1.16 (VDD2)
- net GND: now also C52.2, C9102.1, C?.2, J10.3 (Pin_3), Q21.2 (S), R9101.1, U1.2 (GND1), U1.8 (GND1)
- net IO4: now also R9101.2
- net at D9101.1 (K), R9105.2: now also R9101.1, R9101.2, U1.12 (L)
- net at D9101.2 (K): now also JP?.2 (B), R9101.1, R9101.2, U1.13 (H)
- net at R9105.1: now also JP?.1 (A)
- net IO5: now reaches U5.29 (PA8)
- new net: D2.2 (A), J10.2 (Pin_2), Q21.3 (D)
- new net: Q21.1 (G), R9101.1, R9101.2
- new net: C?.1, R9101.2 (x2)

Commit message: fix prj; description -> Comments
Parts:
- Q1, Q2, Q21: Comments (none) -> bss123; description bss123 -> (none)
Changed lines of the file:
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@@
       (effects (font (size 1.27 1.27)) hide)
     )
-    (property "description" "bss123" (at 237.49 105.41 0)
+    (property "Comments" "bss123" (at 237.49 105.41 0)
       (effects (font (size 1.27 1.27)) hide)
     )
@@
       (effects (font (size 1.27 1.27)) hide)
     )
-    (property "description" "bss123" (at 242.57 189.23 0)
+    (property "Comments" "bss123" (at 242.57 189.23 0)
       (effects (font (size 1.27 1.27)) hide)
     )
@@
       (effects (font (size 1.27 1.27)) hide)
     )
-    (property "description" "bss123" (at 327.66 85.09 0)
+    (property "Comments" "bss123" (at 327.66 85.09 0)
       (effects (font (size 1.27 1.27)) hide)
     )
