File: hardware/main.kicad_pcb (KiCad board)
At the start: 2 copper layers, 66 x 33 mm, 10 parts

Commit message: update prj
Parts:
- added C1: 100n, Capacitor_SMD:C_0603_1608Metric, F.Cu at (154.1, -89.6)
- added C10: 2.2u, Capacitor_SMD:C_1206_3216Metric, F.Cu at (155.0, -54.8)
- added C11: 22u, Capacitor_SMD:C_0805_2012Metric, F.Cu at (160.0, -55.7)
- added C12: 22u, Capacitor_SMD:C_0805_2012Metric, F.Cu at (160.0, -52.7)
- added C13: 100n, Capacitor_SMD:C_0603_1608Metric, F.Cu at (154.1, -77.0)
- added C14: 100n, Capacitor_SMD:C_0603_1608Metric, F.Cu at (154.1, -74.5)
- added C15: 1u, Capacitor_SMD:C_0603_1608Metric, F.Cu at (-115.0, 14.5)
- added C16: 330p, Capacitor_SMD:C_0603_1608Metric, F.Cu at (154.1, -69.5)
- added C17: 330p, Capacitor_SMD:C_0603_1608Metric, F.Cu at (154.1, -67.0)
- added C18: 1u, Capacitor_SMD:C_0603_1608Metric, F.Cu at (-115.0, 22.0)
- added C19: 1u, Capacitor_SMD:C_0603_1608Metric, F.Cu at (-111.0, -3.06)
- added C2: 22u, Capacitor_SMD:C_0805_2012Metric, F.Cu at (160.0, -61.7)
- added C20: 1u, Capacitor_SMD:C_0603_1608Metric, F.Cu at (-111.0, -0.55)
- added C21: 22u, Capacitor_SMD:C_0805_2012Metric, F.Cu at (-79.3, -53.7)
- added C22: 100n, Capacitor_SMD:C_0603_1608Metric, F.Cu at (-3.21, 33.5)
- added C23: 100n, Capacitor_SMD:C_0603_1608Metric, F.Cu at (-3.21, 36.0)
- added C24: 100n, Capacitor_SMD:C_0603_1608Metric, F.Cu at (-3.21, 38.5)
- added C25: 100n, Capacitor_SMD:C_0603_1608Metric, F.Cu at (-3.21, 41.0)
- added C26: 100n, Capacitor_SMD:C_0603_1608Metric, F.Cu at (-3.21, 43.5)
- added C27: 100n, Capacitor_SMD:C_0603_1608Metric, F.Cu at (-3.21, 46.0)
- added C28: 100n, Capacitor_SMD:C_0603_1608Metric, F.Cu at (28.1, -48.0)
- added C29: 10u, Capacitor_SMD:C_0805_2012Metric, F.Cu at (-1.35, 71.4)
- added C3: 100n, Capacitor_SMD:C_0603_1608Metric, F.Cu at (154.1, -87.1)
- added C30: 1u, Capacitor_SMD:C_0603_1608Metric, F.Cu at (-111.0, 19.5)
- added C31: 1n, Capacitor_SMD:C_0603_1608Metric, F.Cu at (-3.21, 53.6)
- added C32: 1u, Capacitor_SMD:C_0603_1608Metric, F.Cu at (0.80, 28.5)
- added C33: 10u, Capacitor_SMD:C_0805_2012Metric, F.Cu at (-1.35, 74.4)
- added C34: 1u, Capacitor_SMD:C_0603_1608Metric, F.Cu at (0.80, 31.0)
- added C35: 1u, Capacitor_SMD:C_0603_1608Metric, F.Cu at (-107.0, 1.96)
- added C36: 100n, Capacitor_SMD:C_0603_1608Metric, F.Cu at (-77.2, -86.1)
- added C37: 1n, Capacitor_SMD:C_0603_1608Metric, F.Cu at (0.80, 38.5)
- added C38: 1u, Capacitor_SMD:C_0603_1608Metric, F.Cu at (-107.0, 9.49)
- added C39: 1u, Capacitor_SMD:C_0603_1608Metric, F.Cu at (0.80, 43.5)
- added C4: 22u, Capacitor_SMD:C_0805_2012Metric, F.Cu at (160.0, -58.7)
- added C40: 10u, Capacitor_SMD:C_0805_2012Metric, F.Cu at (-1.35, 77.4)
- added C41: 1n, Capacitor_SMD:C_0603_1608Metric, F.Cu at (0.80, 46.0)
- added C42: 1u, Capacitor_SMD:C_0603_1608Metric, F.Cu at (-107.0, 17.0)
- added C43: 1u, Capacitor_SMD:C_0603_1608Metric, F.Cu at (0.80, 51.1)
- added C44: 1u, Capacitor_SMD:C_0603_1608Metric, F.Cu at (-107.0, 22.0)
- added C45: 1u, Capacitor_SMD:C_0603_1608Metric, F.Cu at (-103.0, -3.06)
- added C46: 1u, Capacitor_SMD:C_0603_1608Metric, F.Cu at (-103.0, -0.55)
- added C47: 1u, Capacitor_SMD:C_0603_1608Metric, F.Cu at (-103.0, 1.96)
- added C48: 12p, Capacitor_SMD:C_0603_1608Metric, F.Cu at (-73.1, -86.1)
- added C49: 12p, Capacitor_SMD:C_0603_1608Metric, F.Cu at (-73.1, -83.6)
- added C5: 100n, Capacitor_SMD:C_0603_1608Metric, F.Cu at (154.1, -84.5)
- added C50: 1u, Capacitor_SMD:C_0603_1608Metric, F.Cu at (-103.0, 9.49)
- added C51: 100n, Capacitor_SMD:C_1206_3216Metric, F.Cu at (96.5, 43.9)
- added C52: 100n, Capacitor_SMD:C_1206_3216Metric, F.Cu at (96.5, 47.2)
- added C53: 1u, Capacitor_SMD:C_0603_1608Metric, F.Cu at (-103.0, 12.0)
- added C54: 100n, Capacitor_SMD:C_1206_3216Metric, F.Cu at (96.5, 50.5)
- added C55: 100n, Capacitor_SMD:C_1206_3216Metric, F.Cu at (96.5, 53.9)
- added C56: JYC3D332MBF, MAS_Package_nostd:JYC3D332MBF, F.Cu at (2.68, 81.8)
- added C57: 100n, Capacitor_SMD:C_0603_1608Metric, F.Cu at (107.7, 23.3)
- added C58: 100n, Capacitor_SMD:C_0603_1608Metric, F.Cu at (107.7, 25.9)
- added C59: 100n, Capacitor_SMD:C_0603_1608Metric, F.Cu at (107.7, 28.4)
- added C6: 1u, Capacitor_SMD:C_0603_1608Metric, F.Cu at (-115.0, 4.47)
- added C60: 1u, Capacitor_SMD:C_0603_1608Metric, F.Cu at (-103.0, 22.0)
- added C61: 12p, Capacitor_SMD:C_0603_1608Metric, F.Cu at (-69.1, -93.6)
- added C62: 12p, Capacitor_SMD:C_0603_1608Metric, F.Cu at (-69.1, -91.1)
- added C63: 1u, Capacitor_SMD:C_0603_1608Metric, F.Cu at (-99.0, 1.96)
- added C64: 100n, Capacitor_SMD:C_1206_3216Metric, F.Cu at (96.5, 57.2)
- added C65: 100n, Capacitor_SMD:C_1206_3216Metric, F.Cu at (96.5, 60.6)
- added C7: 1u, Capacitor_SMD:C_0603_1608Metric, F.Cu at (-115.0, 6.98)
- added C8: 2.2u, Capacitor_SMD:C_1206_3216Metric, F.Cu at (155.0, -61.5)
- added C9: 2.2u, Capacitor_SMD:C_1206_3216Metric, F.Cu at (155.0, -58.2)
- added D1: 1N4148WS, Diode_SMD:D_SOD-323, F.Cu at (-80.6, 22.5)
- added D10: SMCJ75A, Diode_SMD:D_SMA, F.Cu at (107.9, 71.4)
- added D11: BZT52C3V3, Diode_SMD:D_SOD-323, F.Cu at (164.2, 33.6)
- added D12: BZT52C3V3, Diode_SMD:D_SOD-323, F.Cu at (164.2, 36.5)
- added D13: ER3J, Diode_SMD:D_SMC, F.Cu at (145.3, 19.7)
- added D14: 1N4148WS, Diode_SMD:D_SOD-323, F.Cu at (164.2, 39.5)
- added D15: BZT52C16SQ, Diode_SMD:D_SOD-323, F.Cu at (164.2, 42.5)
- added D16: BZT52C3V3, Diode_SMD:D_SOD-323, F.Cu at (-76.3, 34.3)
- added D17: BZT52C5V6S, Diode_SMD:D_SOD-323, F.Cu at (-97.4, 71.5)
- added D18: BZT52C5V6S, Diode_SMD:D_SOD-323, F.Cu at (-109.3, 71.5)
- added D19: BZT52C5V6S, Diode_SMD:D_SOD-323, F.Cu at (-64.4, 25.8)
- added D2: MBR0540, Diode_SMD:D_SOD-123, F.Cu at (86.0, -60.0)
- added D20: BZT52C5V6S, Diode_SMD:D_SOD-323, F.Cu at (-64.4, 36.1)
- added D21: BZT52C5V6S, Diode_SMD:D_SOD-323, F.Cu at (-73.6, 81.8)
- added D22: BZT52C5V6S, Diode_SMD:D_SOD-323, F.Cu at (-64.4, 15.5)
- added D23: BZT52C5V6S, Diode_SMD:D_SOD-323, F.Cu at (-64.4, 46.4)
- added D24: BZT52C5V6S, Diode_SMD:D_SOD-323, F.Cu at (-85.5, 71.5)
- added D25: BZT52C5V6S, Diode_SMD:D_SOD-323, F.Cu at (-64.4, 56.7)
- added D26: BZT52C5V6S, Diode_SMD:D_SOD-323, F.Cu at (-64.4, 5.18)
- added D27: BZT52C5V6S, Diode_SMD:D_SOD-323, F.Cu at (-64.4, -5.13)
- added D28: BZT52C5V6S, Diode_SMD:D_SOD-323, F.Cu at (-97.4, 81.8)
- added D29: BZT52C5V6S, Diode_SMD:D_SOD-323, F.Cu at (-85.5, 81.8)
- added D3: STPS2L40U, Diode_SMD:D_SMB, F.Cu at (213.8, -82.5)
- added D30: BZT52C5V6S, Diode_SMD:D_SOD-323, F.Cu at (-73.6, 71.5)
- added D31: BZT52C5V6S, Diode_SMD:D_SOD-323, F.Cu at (-109.3, 81.8)
- added D4: PESD1CAN, Package_TO_SOT_SMD:SOT-23, F.Cu at (218.5, -39.4)
- added D5: 1N4148WS, Diode_SMD:D_SOD-323, F.Cu at (-80.6, 25.4)
- added D6: 1N4148WS, Diode_SMD:D_SOD-323, F.Cu at (57.0, 62.2)
- added D7: 1N4148WS, Diode_SMD:D_SOD-323, F.Cu at (-80.6, 31.3)
- added D8: 1N4148WS, Diode_SMD:D_SOD-323, F.Cu at (57.0, 68.1)
- added D9: BZT52C3V3, Diode_SMD:D_SOD-323, F.Cu at (57.0, 71.0)
- added F1: 12T.30000063AG12S1B02, Fuse:Fuse_1206_3216Metric, F.Cu at (220.6, -70.9)
- added F2: S1032-F-40.0A, MAS_Package_nostd:Fuse_1032, F.Cu at (132.6, 14.4)
- added J1: HC-MX3.0-2*4A, MAS_Package_std:Molex_Micro-Fit_3.0_43045-0812_2x04_P3.00mm_Vertical, F.Cu at (-105.0, 39.2)
- added J2: B2B-XH-A, MAS_Package_std:JST_XH_B2B-XH-AM_1x02_P2.50mm_Vertical, F.Cu at (77.5, -44.0)
- added J3: DS1013-10S, Connector_IDC:IDC-Header_2x05_P2.54mm_Vertical, F.Cu at (-47.5, -61.2)
- added J4: HC-MX3.0-2*4A, MAS_Package_std:Molex_Micro-Fit_3.0_43045-0812_2x04_P3.00mm_Vertical, F.Cu at (-105.0, 50.0)
- added J5: B2B-XH-A, MAS_Package_std:JST_XH_B2B-XH-AM_1x02_P2.50mm_Vertical, F.Cu at (4.34, 66.0)
- added J6: B2B-XH-A, MAS_Package_std:JST_XH_B2B-XH-AM_1x02_P2.50mm_Vertical, F.Cu at (4.34, 73.8)
- added J7: IDC-08M, Connector_IDC:IDC-Header_2x04_P2.54mm_Vertical, F.Cu at (-47.5, -38.8)
- added J8: XT60, MAS_Package_nostd:AMASS_XT60-F_1x02_P7.20mm_Vertical, F.Cu at (145.2, 58.9)
- added J9: XT60, MAS_Package_nostd:AMASS_XT60-F_1x02_P7.20mm_Vertical, F.Cu at (145.2, 69.1)
- added JP1: Jload, MAS_Package_nostd:SolderJumper_Open_Pad0.5x0.8mm, F.Cu at (219.2, -78.3)
- added JP2: div1, MAS_Package_nostd:SolderJumper_Open_Pad0.5x0.8mm, F.Cu at (-20.1, -80.1)
- added JP3: div1, MAS_Package_nostd:SolderJumper_Open_Pad0.5x0.8mm, F.Cu at (-20.1, -77.7)
- added L1: SMMS0650-100M, MAS_Package_nostd:SMDL_7.1x6.6x5mm, F.Cu at (203.2, -67.7)
- added Q1: 5N10-MS, Package_TO_SOT_SMD:SOT-23, F.Cu at (91.9, -45.0)
- added Q10: IRLML6402, Package_TO_SOT_SMD:SOT-23, F.Cu at (-74.9, 85.9)
- added Q11: IRLML6402, Package_TO_SOT_SMD:SOT-23, F.Cu at (-65.7, 19.5)
- added Q12: IRLML6402, Package_TO_SOT_SMD:SOT-23, F.Cu at (-65.7, 50.5)
- added Q13: IRLML6402, Package_TO_SOT_SMD:SOT-23, F.Cu at (-86.8, 75.6)
- added Q14: IRLML6402, Package_TO_SOT_SMD:SOT-23, F.Cu at (-65.7, 60.8)
- added Q15: IRLML6402, Package_TO_SOT_SMD:SOT-23, F.Cu at (-65.7, 9.22)
- added Q16: IRLML6402, Package_TO_SOT_SMD:SOT-23, F.Cu at (-65.7, -1.09)
- added Q17: IRLML6402, Package_TO_SOT_SMD:SOT-23, F.Cu at (-98.7, 85.9)
- added Q18: IRLML6402, Package_TO_SOT_SMD:SOT-23, F.Cu at (-86.8, 85.9)
- added Q19: IRLML6402, Package_TO_SOT_SMD:SOT-23, F.Cu at (-74.9, 75.6)
- added Q2: 5N10-MS, Package_TO_SOT_SMD:SOT-23, F.Cu at (57.1, 87.6)
- added Q20: IRLML6402, Package_TO_SOT_SMD:SOT-23, F.Cu at (-110.6, 85.9)
- added Q3: AO3401A, Package_TO_SOT_SMD:SOT-23, F.Cu at (160.1, 69.3)
- added Q4: IPT007N06N, Package_TO_SOT_SMD:Infineon_PG-HSOF-8-1, F.Cu at (120.7, 38.0)
- added Q5: IPT007N06N, Package_TO_SOT_SMD:Infineon_PG-HSOF-8-1, F.Cu at (120.7, 49.6)
- added Q6: IRLML6402, Package_TO_SOT_SMD:SOT-23, F.Cu at (-98.7, 75.6)
- added Q7: IRLML6402, Package_TO_SOT_SMD:SOT-23, F.Cu at (-110.6, 75.6)
- added Q8: IRLML6402, Package_TO_SOT_SMD:SOT-23, F.Cu at (-65.7, 29.8)
- added Q9: IRLML6402, Package_TO_SOT_SMD:SOT-23, F.Cu at (-65.7, 40.1)
- added R1: 100R, Resistor_SMD:R_0603_1608Metric, F.Cu at (170.2, -82.0)
- added R10: 120R, Resistor_SMD:R_1206_3216Metric, F.Cu at (220.6, -67.6)
- added R11: 100R, Resistor_SMD:R_0603_1608Metric, F.Cu at (86.0, -71.2)
- added R12: 100k, Resistor_SMD:R_0603_1608Metric, F.Cu at (86.0, -68.7)
- added R13: 200R, Resistor_SMD:R_0603_1608Metric, F.Cu at (12.8, 36.0)
- added R14: 100k, Resistor_SMD:R_0603_1608Metric, F.Cu at (44.2, -58.1)
- added R15: 100R, Resistor_SMD:R_0603_1608Metric, F.Cu at (12.8, 41.0)
- added R16: 10k, Resistor_SMD:R_0603_1608Metric, F.Cu at (-65.1, -78.6)
- added R17: 10k, Resistor_SMD:R_0603_1608Metric, F.Cu at (-65.1, -76.1)
- added R18: 1M, Resistor_SMD:R_0603_1608Metric, F.Cu at (-65.1, -73.6)
- added R19: 100k, Resistor_SMD:R_0603_1608Metric, F.Cu at (12.8, 51.1)
- added R2: 100k, Resistor_SMD:R_0603_1608Metric, F.Cu at (170.2, -79.5)
- added R20: 5.6k, Resistor_SMD:R_0603_1608Metric, F.Cu at (44.2, -43.0)
- added R21: 1k, Resistor_SMD:R_0603_1608Metric, F.Cu at (-91.0, -3.06)
- added R22: 100R, Resistor_SMD:R_0603_1608Metric, F.Cu at (16.8, 31.0)
- added R23: 100k, Resistor_SMD:R_0603_1608Metric, F.Cu at (16.8, 33.5)
- added R24: 100R, Resistor_SMD:R_0603_1608Metric, F.Cu at (16.8, 36.0)
- added R25: 100R, Resistor_SMD:R_0603_1608Metric, F.Cu at (16.8, 38.5)
- added R26: 4.7k, Resistor_SMD:R_0603_1608Metric, F.Cu at (-61.1, -81.1)
- added R27: 100R, Resistor_SMD:R_0603_1608Metric, F.Cu at (16.8, 43.5)
- added R28: 4.7k, Resistor_SMD:R_0603_1608Metric, F.Cu at (-61.1, -76.1)
- added R29: 10k/NTC, Resistor_SMD:R_0603_1608Metric, F.Cu at (16.8, 48.5)
- added R3: 0R, Resistor_SMD:R_0603_1608Metric, F.Cu at (170.2, -77.0)
- added R30: 1k, Resistor_SMD:R_0603_1608Metric, F.Cu at (-91.0, 19.5)
- added R31: 1k, Resistor_SMD:R_0603_1608Metric, F.Cu at (16.8, 53.6)
- added R32: 4.7k, Resistor_SMD:R_0603_1608Metric, F.Cu at (20.8, 28.5)
- added R33: 4.7k, Resistor_SMD:R_0603_1608Metric, F.Cu at (20.8, 31.0)
- added R34: 51k, Resistor_SMD:R_0603_1608Metric, F.Cu at (20.8, 33.5)
- added R35: 1k, Resistor_SMD:R_0603_1608Metric, F.Cu at (123.8, 13.3)
- added R36: 10M, Resistor_SMD:R_0805_2012Metric, F.Cu at (58.8, 32.0)
- added R37: 1M, Resistor_SMD:R_0603_1608Metric, F.Cu at (123.8, 15.8)
- added R38: 100R, Resistor_SMD:R_0603_1608Metric, F.Cu at (123.8, 18.3)
- added R39: 100R, Resistor_SMD:R_0603_1608Metric, F.Cu at (123.8, 20.8)
- added R4: 47k, Resistor_SMD:R_0603_1608Metric, F.Cu at (170.2, -74.5)
- added R40: 1M, Resistor_SMD:R_0603_1608Metric, F.Cu at (123.8, 23.3)
- added R41: 1M, Resistor_SMD:R_0603_1608Metric, F.Cu at (123.8, 25.9)
- added R42: 3m, Resistor_SMD:R_2512_6332Metric, F.Cu at (155.0, 18.3)
- added R43: 1k, Resistor_SMD:R_0603_1608Metric, F.Cu at (-87.0, 19.5)
- added R44: 3m, Resistor_SMD:R_2512_6332Metric, F.Cu at (155.0, 23.2)
- added R45: 1k, Resistor_SMD:R_0603_1608Metric, F.Cu at (-103.1, 74.6)
- added R46: 10k, Resistor_SMD:R_0603_1608Metric, F.Cu at (-103.1, 77.1)
- added R47: 100R, Resistor_SMD:R_1206_3216Metric, F.Cu at (-102.3, 71.7)
- added R48: 1k, Resistor_SMD:R_0603_1608Metric, F.Cu at (-115.0, 74.6)
- added R49: 10k, Resistor_SMD:R_0603_1608Metric, F.Cu at (-115.0, 77.1)
- added R5: 18k, Resistor_SMD:R_0603_1608Metric, F.Cu at (170.2, -72.0)
- added R50: 100R, Resistor_SMD:R_1206_3216Metric, F.Cu at (-114.2, 71.7)
- added R51: 1k, Resistor_SMD:R_0603_1608Metric, F.Cu at (-70.2, 28.9)
- added R52: 10k, Resistor_SMD:R_0603_1608Metric, F.Cu at (-70.2, 31.4)
- added R53: 100R, Resistor_SMD:R_1206_3216Metric, F.Cu at (-69.4, 26.0)
- added R54: 1k, Resistor_SMD:R_0603_1608Metric, F.Cu at (-70.2, 39.2)
- added R55: 10k, Resistor_SMD:R_0603_1608Metric, F.Cu at (-70.2, 41.7)
- added R56: 100R, Resistor_SMD:R_1206_3216Metric, F.Cu at (-69.4, 36.3)
- added R57: 1k, Resistor_SMD:R_0603_1608Metric, F.Cu at (-79.3, 84.9)
- added R58: 10k, Resistor_SMD:R_0603_1608Metric, F.Cu at (-79.3, 87.4)
- added R59: 100R, Resistor_SMD:R_1206_3216Metric, F.Cu at (-78.5, 82.0)
- added R6: 0R, Resistor_SMD:R_0603_1608Metric, F.Cu at (170.2, -69.5)
- added R60: 1k, Resistor_SMD:R_0603_1608Metric, F.Cu at (-70.2, 18.6)
- added R61: 10k, Resistor_SMD:R_0603_1608Metric, F.Cu at (-70.2, 21.1)
- added R62: 100R, Resistor_SMD:R_1206_3216Metric, F.Cu at (-69.4, 15.7)
- added R63: 1k, Resistor_SMD:R_0603_1608Metric, F.Cu at (-70.2, 49.5)
- added R64: 10k, Resistor_SMD:R_0603_1608Metric, F.Cu at (-70.2, 52.0)
- added R65: 100R, Resistor_SMD:R_1206_3216Metric, F.Cu at (-69.4, 46.6)
- added R66: 1k, Resistor_SMD:R_0603_1608Metric, F.Cu at (-91.2, 74.6)
- added R67: 10k, Resistor_SMD:R_0603_1608Metric, F.Cu at (-91.2, 77.1)
- added R68: 100R, Resistor_SMD:R_1206_3216Metric, F.Cu at (-90.4, 71.7)
- added R69: 1k, Resistor_SMD:R_0603_1608Metric, F.Cu at (-70.2, 59.8)
- added R7: 18k, Resistor_SMD:R_0603_1608Metric, F.Cu at (170.2, -67.0)
- added R70: 10k, Resistor_SMD:R_0603_1608Metric, F.Cu at (-70.2, 62.3)
- added R71: 100R, Resistor_SMD:R_1206_3216Metric, F.Cu at (-69.4, 56.9)
- added R72: 1k, Resistor_SMD:R_0603_1608Metric, F.Cu at (-70.2, 8.25)
- added R73: 10k, Resistor_SMD:R_0603_1608Metric, F.Cu at (-70.2, 10.8)
- added R74: 100R, Resistor_SMD:R_1206_3216Metric, F.Cu at (-69.4, 5.35)
- added R75: 1k, Resistor_SMD:R_0603_1608Metric, F.Cu at (-70.2, -2.06)
- added R76: 10k, Resistor_SMD:R_0603_1608Metric, F.Cu at (-70.2, 0.45)
- added R77: 100R, Resistor_SMD:R_1206_3216Metric, F.Cu at (-69.4, -4.96)
- added R78: 1k, Resistor_SMD:R_0603_1608Metric, F.Cu at (-103.1, 84.9)
- added R79: 10k, Resistor_SMD:R_0603_1608Metric, F.Cu at (-103.1, 87.4)
- added R8: 100R, Resistor_SMD:R_0603_1608Metric, F.Cu at (170.2, -64.5)
- added R80: 100R, Resistor_SMD:R_1206_3216Metric, F.Cu at (-102.3, 82.0)
- added R81: 1k, Resistor_SMD:R_0603_1608Metric, F.Cu at (-91.2, 84.9)
- added R82: 10k, Resistor_SMD:R_0603_1608Metric, F.Cu at (-91.2, 87.4)
- added R83: 100R, Resistor_SMD:R_1206_3216Metric, F.Cu at (-90.4, 82.0)
- added R84: 1k, Resistor_SMD:R_0603_1608Metric, F.Cu at (-79.3, 74.6)
- added R85: 10k, Resistor_SMD:R_0603_1608Metric, F.Cu at (-79.3, 77.1)
- added R86: 100R, Resistor_SMD:R_1206_3216Metric, F.Cu at (-78.5, 71.7)
- added R87: 1k, Resistor_SMD:R_0603_1608Metric, F.Cu at (-115.0, 84.9)
- added R88: 10k, Resistor_SMD:R_0603_1608Metric, F.Cu at (-115.0, 87.4)
- added R89: 100R, Resistor_SMD:R_1206_3216Metric, F.Cu at (-114.2, 82.0)
- added R9: 100R, Resistor_SMD:R_0603_1608Metric, F.Cu at (174.2, -89.6)
- added SW1: TS-1187A-B-A-B, Button_Switch_SMD:SW_SPST_TL3342, F.Cu at (15.1, 96.0)
- added TP1: SCL, MAS_Package_std:TestPoint_Pad_D0.5mm, F.Cu at (57.5, 34.4)
- added TP2: SDA, MAS_Package_std:TestPoint_Pad_D0.5mm, F.Cu at (57.5, 36.1)
- added U1: AM1LS-0505S-NZ, MAS_Package_nostd:Converter_DCDC_Aimtec_AM1LS_SMD, F.Cu at (179.1, -32.6)
- added U2: LMR16030SDDAR, MAS_Package_std:SOIC-8-1EP_3.9x4.9mm_P1.27mm_EP2.29x3mm, F.Cu at (166.5, -29.4)
- added U3: CA-IS3050G, MAS_Package_std:SOIC-8_7.5x5.85mm_P1.27mm, F.Cu at (191.2, -87.1)
- added U4: BQ7694003DBT, Package_SO:TSSOP-44_4.4x11.2mm_P0.5mm, F.Cu at (-48.0, 5.00)
- added U5: STM32F103C8Tx, Package_QFP:LQFP-48_7x7mm_P0.5mm, F.Cu at (-44.8, -85.2)
- added Y1: NX3215SA-32.768, MAS_Package_std:Crystal_SMD_3215-2Pin_3.2x1.5mm, F.Cu at (-18.8, -93.2)
- added Y2: X50328MSB2GI, MAS_Package_std:Crystal_SMD_5032-2Pin_5.0x3.2mm, F.Cu at (-26.6, -71.3)
- moved FID1 34.4 mm to (96.0, -35.0)
- moved FID4 34.4 mm to (96.0, -35.0)
- moved H2 34.4 mm to (96.0, -29.0)
- moved H3 34.4 mm to (96.0, -9.00)
- moved FID2 5.00 mm to (4.00, -35.0)
- moved FID3 5.00 mm to (4.00, -15.0)
- moved FID5 5.00 mm to (4.00, -15.0)
- moved FID6 5.00 mm to (4.00, -35.0)
- moved H1 5.00 mm to (4.00, -9.00)
- moved H4 5.00 mm to (4.00, -29.0)
Connections:
- H4 pad 1: (no net) -> GNDREF
Other:
- board size 66 x 33 mm -> 100 x 38 mm

Commit message: update pcb
Parts:
- J7: footprint Connector_IDC:IDC-Header_2x04_P2.54mm_Vertical -> Connector_PinSocket_1.27mm:PinSocket_2x04_P1.27mm_Vertical
- JP2: value div1 -> BOOT
- JP3: value div1 -> PWRprog
- moved R88 250.5 mm to (114.3, -13.3), turned to 90 degrees
- moved R87 248.0 mm to (112.6, -13.3), turned to 90 degrees
- moved R89 243.1 mm to (113.4, -3.17), turned to -90 degrees
- moved Q20 242.7 mm to (113.4, -7.62), turned to -90 degrees
- moved D31 241.2 mm to (113.4, -10.8)
- moved R79 229.3 mm to (102.9, -13.3), turned to 90 degrees
- moved R78 226.7 mm to (101.2, -13.3), turned to 90 degrees
- moved R82 222.1 mm to (106.7, -13.3), turned to 90 degrees
- moved Q17 221.4 mm to (102.0, -7.62), turned to -90 degrees
- moved R80 221.4 mm to (102.0, -3.17), turned to -90 degrees
- moved C60 220.7 mm to (114.3, -16.5), turned to 90 degrees
- moved D28 219.8 mm to (102.0, -10.8)
- moved R81 219.5 mm to (105.0, -13.3), turned to 90 degrees
- moved C53 216.3 mm to (111.5, -15.9)
- moved C63 214.4 mm to (114.3, -19.7), turned to 90 degrees
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Other:
- board size 100 x 38 mm -> 158 x 38 mm

Commit message: update readme
Parts:
- J1, J4: value HC-MX3.0-2*4A -> IDC-08M; footprint MAS_Package_std:Molex_Micro-Fit_3.0_43045-0812_2x04_P3.00mm_Vertical -> Connector_IDC:IDC-Header_2x04_P2.54mm_Vertical
- J2: value B2B-XH-A -> B3B-XH-A; footprint MAS_Package_std:JST_XH_B2B-XH-AM_1x02_P2.50mm_Vertical -> MAS_Package_std:JST_XH_B3B-XH-AM_1x03_P2.50mm_Vertical
- moved J4 7.69 mm to (59.9, -6.10), turned to 180 degrees
- moved J1 7.61 mm to (96.5, -6.10), turned to 180 degrees
- moved J7 1.91 mm to (15.9, -33.0)
- moved JP3 1.91 mm to (10.2, -33.5)
- moved C18 1.60 mm to (58.8, -20.3)
- moved C46 0.97 mm to (95.6, -20.3)

Commit message: update can
Parts:
- removed U3: CA-IS3050G, MAS_Package_std:SOIC-8_7.5x5.85mm_P1.27mm
- added D32: MBR0540, Diode_SMD:D_SOD-123, F.Cu at (12.7, -45.7)
- added J10: B3B-XH-A, MAS_Package_std:JST_XH_B3B-XH-AM_1x03_P2.50mm_Vertical, F.Cu at (12.0, -50.1)
- added Q21: 5N10-MS, Package_TO_SOT_SMD:SOT-23, F.Cu at (6.35, -43.5)
- added R90: 100R, Resistor_SMD:R_0603_1608Metric, F.Cu at (8.89, -45.2)
- added R91: 100k, Resistor_SMD:R_0603_1608Metric, F.Cu at (6.35, -46.3)
- C14: value 100n -> 1n (-); footprint Capacitor_SMD:C_0603_1608Metric -> Capacitor_SMD:C_1206_3216Metric
- C2: value 22u -> 10u; footprint Capacitor_SMD:C_0805_2012Metric -> Capacitor_SMD:C_0603_1608Metric
- C4: value 22u -> 100n; footprint Capacitor_SMD:C_0805_2012Metric -> Capacitor_SMD:C_0603_1608Metric
- C5: value 100n -> 10u
- U1: value AM1LS-0505S-NZ -> CA-IS3062W; footprint MAS_Package_nostd:Converter_DCDC_Aimtec_AM1LS_SMD -> Package_SO:SOIC-16W_7.5x10.3mm_P1.27mm
- moved C28 66.1 mm to (49.5, -22.4)
- moved R14 66.1 mm to (47.6, -22.4)
- moved R20 66.1 mm to (51.4, -22.4)
- moved JP1 45.9 mm to (39.4, -49.3)
- moved C16 45.9 mm to (36.2, -51.8)
- moved C17 45.9 mm to (34.6, -51.8)
- moved D4 45.9 mm to (39.4, -54.8)
- moved R10 45.9 mm to (39.4, -51.4)
- moved R3 45.9 mm to (41.3, -48.3), turned to 90 degrees
- moved R6 45.9 mm to (37.5, -48.3)
- moved R8 45.9 mm to (36.2, -54.8)
- moved R9 45.9 mm to (34.6, -54.8)
- moved L1 42.1 mm to (70.7, -63.3), turned to 0 degrees
- moved C13 39.2 mm to (74.5, -57.9), turned to -90 degrees
- moved C9 39.0 mm to (51.7, -64.9), turned to 90 degrees
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Connections:
- C1 pad 1: +5V -> /CANvcc
- C1 pad 2: GND -> /CANgnd
- C14 pad 1: +3.3V -> GND
- C14 pad 2: GND -> /CANgnd
- C2 pad 1: +5V -> /CANvcc
- C2 pad 2: GND -> /CANgnd
- C4 pad 1: /CANvcc -> +3.3V
- C4 pad 2: /CANgnd -> GND
- C5 pad 1: /CANvcc -> +3.3V
- C5 pad 2: /CANgnd -> GND
- D4 pad 1: Net-(U3-CANL) -> Net-(U1-L)
- R10 pad 2: Net-(U3-CANL) -> Net-(U1-L)
- R3 pad 1: Net-(JP1-B) -> /CANH
- R3 pad 2: /CANH -> Net-(JP1-B)
- R6 pad 2: Net-(U3-CANL) -> Net-(U1-L)
- R8 pad 1: Net-(U3-CANL) -> Net-(U1-L)
- U1 pad 1: GND -> +3.3V
- U1 pad 2: +5V -> GND
- U1 pad 4: /CANgnd -> unconnected-(U1-NC-Pad4)
- U1 pad 5: /CANvcc -> /CANrx
- U1 pad 8: unconnected-(U1-NC-Pad8) -> GND
- U5 pad 29: unconnected-(U5-PA8-Pad29) -> /IO5
